File: pcb/_autosave-OpenNixie.kicad_pcb (KiCad board)
At the start: 2 copper layers, 137 parts, among them J1 Conn_01x02_Female, J10 Conn_01x10_Female, J2 Conn_01x03_Female, J3 Conn_01x03_Female, J4 DC 12V, J5 Conn_01x04_Female, J6 Conn_01x03_Female, J7 Conn_01x10_Female, J8 Conn_01x10_Female, J9 Conn_01x10_Female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

Commit message: Lint & Schematic update
Parts:
- BT1: value CR2032 -> 3V
