File: pcb/OpenNixie.kicad_pcb (KiCad board)
At the start: 2 copper layers, 137 parts, among them J1 Conn_01x02_Female, J10 Conn_01x10_Female, J2 Conn_01x03_Female, J3 Conn_01x03_Female, J4 DC 12V, J5 Conn_01x04_Female, J6 Conn_01x03_Female, J7 Conn_01x10_Female, J8 Conn_01x10_Female, J9 Conn_01x10_Female, Q1 S8050, Q10 MPSA42, Q11 MPSA42, Q12 MPSA42, Q13 MPSA42, Q14 MPSA42, Q15 MPSA42, Q16 MPSA42, Q17 MPSA42, Q18 MPSA42, Q19 MPSA42, Q2 IRFU4620, Q20 MPSA42, Q21 MPSA42, Q22 MPSA42, Q23 MPSA42, Q24 MPSA42, Q25 MPSA42, Q26 MPSA42, Q27 MPSA42, Q28 MPSA42, Q29 MPSA42, Q3 MPSA42, Q30 MPSA42, Q31 MPSA42, Q32 MPSA42, Q33 MPSA42, Q34 MPSA42, Q35 MPSA42, Q36 MPSA42, Q37 MPSA42, Q38 MPSA42, Q39 MPSA42, Q4 MPSA42, Q40 MPSA42, Q41 MPSA42, Q42 MPSA42, Q5 MPSA42, Q6 MPSA42, Q7 MPSA42, Q8 MPSA42, Q9 MPSA42, SW1 SW_SPST, U1 LM7805_TO220, U10 74LS138, U11 74LS138, U12 74LS138, U13 74LS138, U14 74HC595, U15 74LS138, U16 74LS138, U2 NE555P, U3 MAX1771CSA, U4 DS3231M, U5 24LC16, U6 TSDP341xx, U7 74LS138, U8 74LS138, U9 74HC595

Commit message: Schematic update
Parts:
- BT1: value CR2032 -> 3V
- J1: footprint Connector_PinHeader_2.54mm:PinHeader_1x02_P2.54mm_Vertical -> Connector_PinSocket_2.54mm:PinSocket_1x02_P2.54mm_Vertical
- J10, J7, J8, J9: footprint Connector_PinHeader_2.54mm:PinHeader_1x10_P2.54mm_Vertical -> Connector_PinSocket_2.54mm:PinSocket_1x10_P2.54mm_Vertical
- J2, J3, J6: footprint Connector_PinHeader_2.54mm:PinHeader_1x03_P2.54mm_Vertical -> Connector_PinSocket_2.54mm:PinSocket_1x03_P2.54mm_Vertical
- J5: footprint Connector_PinHeader_2.54mm:PinHeader_1x04_P2.54mm_Vertical -> Connector_PinSocket_2.54mm:PinSocket_1x04_P2.54mm_Vertical
- Q2: value IRFU4620 -> IRFB4620; footprint Package_TO_SOT_THT:TO-251-3-1EP_Horizontal_TabDown -> Package_TO_SOT_THT:TO-220-3_Horizontal_TabDown
- R6: value 1k -> 20k
- moved U11 214.0 mm to (32.7, -26.9)
- moved U14 213.2 mm to (36.3, -44.7), turned to 90 degrees
- moved U8 209.5 mm to (45.3, -26.7)
- moved U9 200.1 mm to (84.7, -38.1)
- moved U13 162.1 mm to (246.5, -24.8)
- moved U7 154.3 mm to (265.7, 17.6)
- moved U15 154.0 mm to (176.1, -24.8)
- moved U12 96.0 mm to (143.2, 25.8), turned to 90 degrees
- moved U10 80.2 mm to (249.4, 29.9)
- moved U16 76.4 mm to (174.9, 25.3), turned to 90 degrees
- moved Q2 67.9 mm to (256.0, 174.4)
- moved U4 49.2 mm to (189.7, 135.1)
- moved J9 26.4 mm to (202.9, 98.6)
- moved BT1 21.4 mm to (177.0, 120.3)
Connections:
- Q2 pad 1: Net-(C6-Pad1) -> Net-(Q2-Pad1)
- Q2 pad 2: Net-(Q2-Pad2) -> Net-(C6-Pad1)
- U12 pad 5: /595_1_P3 -> GND
- U13 pad 5: /595_1_P7 -> GND
- U3 pad 1: Net-(Q2-Pad2) -> Net-(Q2-Pad1)
- U7 pad 5: /595_0_P3 -> GND
- U8 pad 5: /595_0_P7 -> GND
