File: pcb/OpenNixie.sch (KiCad schematic (older format))
At the start: 136 parts, among them J1 Conn_01x02_Female, J10 Conn_01x10_Female, J2 Conn_01x03_Female, J3 Conn_01x03_Female, J4 DC 12V, J5 Conn_01x04_Female, J6 Conn_01x03_Female, J7 Conn_01x10_Female, J8 Conn_01x10_Female, J9 Conn_01x10_Female, Q1 S8050, Q10 MPSA42, Q11 MPSA42, Q12 MPSA42, Q13 MPSA42, Q14 MPSA42, Q15 MPSA42, Q16 MPSA42, Q17 MPSA42, Q18 MPSA42, Q19 MPSA42, Q2 IRFU4620, Q20 MPSA42, Q21 MPSA42, Q22 MPSA42, Q23 MPSA42, Q24 MPSA42, Q25 MPSA42, Q26 MPSA42, Q27 MPSA42, Q28 MPSA42, Q29 MPSA42, Q3 MPSA42, Q30 MPSA42, Q31 MPSA42, Q32 MPSA42, Q33 MPSA42, Q34 MPSA42, Q35 MPSA42, Q36 MPSA42, Q37 MPSA42, Q38 MPSA42, Q39 MPSA42, Q4 MPSA42, Q40 MPSA42, Q41 MPSA42, Q42 MPSA42, Q5 MPSA42, Q6 MPSA42, Q7 MPSA42, Q8 MPSA42, Q9 MPSA42, U1 LM7805_TO220, U10 74LS138, U11 74LS138, U12 74LS138, U13 74LS138, U14 74HC595, U15 74LS138, U16 74LS138, U2 NE555P, U3 MAX1771CPA, U4 DS3231M, U5 24LC16, U6 TSDP341xx, U7 74LS138, U8 74LS138, U9 74HC595

Commit message: Lint & Schematic update
Parts:
- removed U3: MAX1771CPA, Package_DIP:DIP-8_W7.62mm, symbol Nixie_Clock:MAX1771CPA
- added SW1: SW_SPST, Button_Switch_THT:SW_DIP_SPSTx01_Slide_9.78x4.72mm_W7.62mm_P2.54mm, symbol Switch:SW_SPST
- added U3: MAX1771CSA, Package_SO:SOIC-8-1EP_3.9x4.9mm_P1.27mm_EP2.29x3mm, symbol Nixie_Clock:MAX1771CSA
- BT1: value CR2302 -> 3V; footprint (none) -> Battery:BatteryHolder_Keystone_1058_1x2032
- C1, C2, C7: footprint (none) -> Capacitor_THT:CP_Radial_D5.0mm_P2.50mm
- C3, C5: footprint (none) -> Capacitor_THT:CP_Radial_D8.0mm_P3.50mm
- C4, C8: footprint (none) -> Capacitor_THT:C_Disc_D3.0mm_W2.0mm_P2.50mm
- C6: footprint (none) -> Capacitor_THT:C_Disc_D3.0mm_W1.6mm_P2.50mm
- D2: footprint (none) -> Diode_SMD:D_SMA
- D3: footprint (none) -> LED_THT:LED_D5.0mm-4_RGB
- J1: footprint (none) -> Connector_PinHeader_2.54mm:PinHeader_1x02_P2.54mm_Vertical
- J10, J7, J8, J9: footprint (none) -> Connector_PinHeader_2.54mm:PinHeader_1x10_P2.54mm_Vertical
- J2, J3, J6: footprint (none) -> Connector_PinHeader_2.54mm:PinHeader_1x03_P2.54mm_Vertical
- J4: footprint (none) -> Connector_BarrelJack:BarrelJack_Horizontal
- J5: footprint (none) -> Connector_PinHeader_2.54mm:PinHeader_1x04_P2.54mm_Vertical
- L1: footprint (none) -> Inductor_THT:L_Radial_D7.0mm_P3.00mm
- R1, R10, R11, R13, R2, R3, R4, R5, R6, R7, R8, R9: footprint (none) -> Resistor_THT:R_Axial_DIN0204_L3.6mm_D1.6mm_P7.62mm_Horizontal
- R12: value 73.2k -> 68k; footprint (none) -> Resistor_THT:R_Axial_DIN0204_L3.6mm_D1.6mm_P7.62mm_Horizontal
- R14: footprint (none) -> Resistor_THT:R_Axial_DIN0207_L6.3mm_D2.5mm_P10.16mm_Horizontal
- R15, R16, R17, R18, R19, R20, R21, R22, R23, R24, R25, R26, R27, R28, R29, R30, R31, R32, R33, R34, R35, R36, R37, R38, R39, R40, R41, R42, R43, R44, R45, R46, R47, R48, R49, R50, R51, R52, R53, R54: value 33k -> 47k; footprint (none) -> Resistor_THT:R_Axial_DIN0204_L3.6mm_D1.6mm_P7.62mm_Horizontal
- RV1: footprint (none) -> Potentiometer_THT:Potentiometer_Vishay_T73YP_Vertical
- U10, U11, U12, U13, U14, U15, U16, U7, U8, U9: footprint (none) -> Package_DIP:DIP-16_W7.62mm
- U5: footprint (none) -> Package_DIP:DIP-8_W7.62mm
Connections:
- net +12V: now also SW1.1 (A), U3.2 (VCC); no longer J4.1
- net GND: now also U3.6 (AGND), U3.7 (GND)
- net SHDN_PIN: now also U3.4 (SHDN)
- net at Q2.2 (G): now also U3.1 (EXT)
- net at R12.1, R5.1: now also U3.3 (FB)
- net at C8.1: now also U3.5 (REF)
- net at Q2.3 (S), R14.1: now also U3.8 (CS)
- new net: J4.1, SW1.2 (B)
Other:
- moved on the sheet: BT1, C1, C2, J4, U1

Commit message: Schematic update
Parts:
- removed Q2: IRFU4620, Package_TO_SOT_THT:TO-251-3-1EP_Horizontal_TabDown, symbol Nixie_Clock:IRFU4620
- added Q2: IRFB4620, Package_TO_SOT_THT:TO-220-3_Horizontal_TabDown, symbol Nixie_Clock:IRFB4620
- J1: footprint Connector_PinHeader_2.54mm:PinHeader_1x02_P2.54mm_Vertical -> Connector_PinSocket_2.54mm:PinSocket_1x02_P2.54mm_Vertical
- J10, J7, J8, J9: footprint Connector_PinHeader_2.54mm:PinHeader_1x10_P2.54mm_Vertical -> Connector_PinSocket_2.54mm:PinSocket_1x10_P2.54mm_Vertical
- J2, J3, J6: footprint Connector_PinHeader_2.54mm:PinHeader_1x03_P2.54mm_Vertical -> Connector_PinSocket_2.54mm:PinSocket_1x03_P2.54mm_Vertical
- J5: footprint Connector_PinHeader_2.54mm:PinHeader_1x04_P2.54mm_Vertical -> Connector_PinSocket_2.54mm:PinSocket_1x04_P2.54mm_Vertical
- R6: value 1k -> 20k
Connections:
- net 595_0_P3: no longer U7.5 (E2)
- net 595_0_P7: no longer U8.5 (E2)
- net 595_1_P3: no longer U12.5 (E2)
- net 595_1_P7: no longer U13.5 (E2)
- net GND: now also U12.5 (E2), U13.5 (E2), U7.5 (E2), U8.5 (E2)
- net at C6.1, D2.2 (A), L1.2: now also Q2.2 (D)
- net at U3.1 (EXT): now also Q2.1 (G)
- net at R14.1, U3.8 (CS): now also Q2.3 (S)
Other:
- moved on the sheet: BT1, C1, C2, C3, C4, C5, C6, C7, C8, D1, D2, D3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
