File: pcb/holder/IN12/IN12.kicad_pcb (KiCad board)
At the start: 2 copper layers, 22.4 x 22.2 mm, 2 parts, among them J1 Nixie_Conn_12P

Commit message: Ver 3.0
Routing:
- net P4: track 13.5 -> 23.8 mm
- net P3: track 7.56 -> 16.7 mm
- net P1: track 5.46 -> 8.04 mm
- net P7: track 5.46 -> 7.84 mm
- net P9: track 7.56 -> 9.10 mm
- net P6: track 12.2 -> 10.7 mm
- net P5: track 13.9 -> 15.3 mm
- net PA: track 20.9 -> 19.5 mm
Changed lines of the file:
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@@
     (pad "1" thru_hole circle (at -4 2.54) (size 1.524 1.524) (drill 0.762) (layers "*.Cu" "*.Mask")
       (net 2 "P1") (pinfunction "1") (pintype "bidirectional"))
-    (pad "2" thru_hole circle (at -2.54 4.5) (size 1.524 1.524) (drill 0.762) (layers "*.Cu" "*.Mask")
+    (pad "2" thru_hole circle (at -2.54 5) (size 1.524 1.524) (drill 0.762) (layers "*.Cu" "*.Mask")
       (net 3 "P2") (pinfunction "2") (pintype "bidirectional"))
-    (pad "3" thru_hole circle (at 0 4.5) (size 1.524 1.524) (drill 0.762) (layers "*.Cu" "*.Mask")
+    (pad "3" thru_hole circle (at 0 5) (size 1.524 1.524) (drill 0.762) (layers "*.Cu" "*.Mask")
       (net 4 "P3") (pinfunction "3") (pintype "passive"))
-    (pad "4" thru_hole circle (at 2.54 4.5) (size 1.524 1.524) (drill 0.762) (layers "*.Cu" "*.Mask")
+    (pad "4" thru_hole circle (at 2.54 5) (size 1.524 1.524) (drill 0.762) (layers "*.Cu" "*.Mask")
       (net 5 "P4") (pinfunction "4") (pintype "bidirectional"))
     (pad "5" thru_hole circle (at 4 2.54) (size 1.524 1.524) (drill 0.762) (layers "*.Cu" "*.Mask")
@@
     (pad "7" thru_hole circle (at 4 -2.54) (size 1.524 1.524) (drill 0.762) (layers "*.Cu" "*.Mask")
       (net 8 "P7") (pinfunction "7") (pintype "bidirectional"))
-    (pad "8" thru_hole circle (at 2.54 -4.5) (size 1.524 1.524) (drill 0.762) (layers "*.Cu" "*.Mask")
+    (pad "8" thru_hole circle (at 2.54 -5) (size 1.524 1.524) (drill 0.762) (layers "*.Cu" "*.Mask")
       (net 9 "P8") (pinfunction "8") (pintype "bidirectional"))
-    (pad "9" thru_hole circle (at 0 -4.5) (size 1.524 1.524) (drill 0.762) (layers "*.Cu" "*.Mask")
+    (pad "9" thru_hole circle (at 0 -5) (size 1.524 1.524) (drill 0.762) (layers "*.Cu" "*.Mask")
       (net 10 "P9") (pinfunction "9") (pintype "bidirectional"))
-    (pad "10" thru_hole circle (at -2.54 -4.5) (size 1.524 1.524) (drill 0.762) (layers "*.Cu" "*.Mask")
+    (pad "10" thru_hole circle (at -2.54 -5) (size 1.524 1.524) (drill 0.762) (layers "*.Cu" "*.Mask")
       (net 11 "unconnected-(J1-Pad10)") (pinfunction "10") (pintype "bidirectional+no_connect"))
     (pad "A" thru_hole circle (at -4 -2.54) (size 1.524 1.524) (drill 0.762) (layers "*.Cu" "*.Mask")
@@
   (gr_rect (start 136.144 88.392) (end 158.496 110.617)
     (stroke (width 0.1) (type default)) (fill none) (layer "Edge.Cuts"))
-  (segment (start 149.102851 101.7016) (end 145.5256 101.7016) (width 0.25) (layer "B.Cu") (net 1))
-  (segment (start 145.5256 101.7016) (end 143.32 99.496) (width 0.25) (layer "B.Cu") (net 1))
-  (segment (start 152.92 103.996) (end 151.397251 103.996) (width 0.25) (layer "B.Cu") (net 1))
-  (segment (start 151.397251 103.996) (end 149.102851 101.7016) (width 0.25) (layer "B.Cu") (net 1))
-  (segment (start 143.32 102.036) (end 143.32 107.496) (width 0.25) (layer "F.Cu") (net 2))
-  (segment (start 144.78 103.996) (end 141.72 103.996) (width 0.25) (layer "B.Cu") (net 3))
-  (segment (start 143.907 100.583) (end 142.707 100.583) (width 0.25) (layer "F.Cu") (net 4))
-  (segment (start 147.32 103.996) (end 143.907 100.583) (width 0.25) (layer "F.Cu") (net 4))
-  (segment (start 142.707 100.583) (end 141.62 99.496) (width 0.25) (layer "F.Cu") (net 4))
-  (segment (start 144.526 99.35365) (end 144.526 96.6216) (width 0.25) (layer "F.Cu") (net 5))
-  (segment (start 149.16835 103.996) (end 144.526 99.35365) (width 0.25) (layer "F.Cu") (net 5))
-  (segment (start 149.86 103.996) (end 149.16835 103.996) (width 0.25) (layer "F.Cu") (net 5))
-  (segment (start 144.526 96.6216) (end 142.9004 94.996) (width 0.25) (layer "F.Cu") (net 5))
-  (segment (start 142.9004 94.996) (end 141.72 94.996) (width 0.25) (layer "F.Cu") (net 5))
-  (segment (start 150.233 100.949) (end 151.32 102.036) (width 0.25) (layer "B.Cu") (net 6))
-  (segment (start 146.233 94.409) (end 146.233 95.7378) (width 0.25) (layer "B.Cu") (net 6))
-  (segment (start 143.32 91.496) (end 146.233 94.409) (width 0.25) (layer "B.Cu") (net 6))
-  (segment (start 150.233 99.7378) (end 150.233 100.949) (width 0.25) (layer "B.Cu") (net 6))
-  (segment (start 146.233 95.7378) (end 150.233 99.7378) (width 0.25) (layer "B.Cu") (net 6))
-  (segment (start 146.233 91.583) (end 147.32 90.496) (width 0.25) (layer "F.Cu") (net 7))
-  (segment (start 146.233 95.48663) (end 146.233 91.583) (width 0.25) (layer "F.Cu") (net 7))
-  (segment (start 150.24237 99.496) (end 146.233 95.48663) (width 0.25) (layer "F.Cu") (net 7))
-  (segment (start 151.32 99.496) (end 150.24237 99.496) (width 0.25) (layer "F.Cu") (net 7))
-  (segment (start 151.32 96.956) (end 151.32 91.496) (width 0.25) (layer "F.Cu") (net 8))
-  (segment (start 149.86 94.996) (end 152.92 94.996) (width 0.25) (layer "B.Cu") (net 9))
-  (segment (start 150.733 98.409) (end 151.933 98.409) (width 0.25) (layer "F.Cu") (net 10))
-  (segment (start 151.933 98.409) (end 153.02 99.496) (width 0.25) (layer "F.Cu") (net 10))
-  (segment (start 147.32 94.996) (end 150.733 98.409) (width 0.25) (layer "F.Cu") (net 10))
-  (segment (start 140.7668 98.43157) (end 140.7668 104.2924) (width 0.25) (layer "B.Cu") (net 12))
-  (segment (start 142.24237 96.956) (end 140.7668 98.43157) (width 0.25) (layer "B.Cu") (net 12))
-  (segment (start 143.32 96.956) (end 142.24237 96.956) (width 0.25) (layer "B.Cu") (net 12))
-  (segment (start 150.4532 106.6292) (end 151.32 107.496) (width 0.25) (layer "B.Cu") (net 12))
-  (segment (start 143.1036 106.6292) (end 150.4532 106.6292) (width 0.25) (layer "B.Cu") (net 12))
-  (segment (start 140.7668 104.2924) (end 143.1036 106.6292) (width 0.25) (layer "B.Cu") (net 12))
+  (segment (start 151.972 103.048) (end 152.92 103.996) (width 0.1) (layer "F.Cu") (net 1))
+  (segment (start 143.32 99.496) (end 146.872 103.048) (width 0.1) (layer "F.Cu") (net 1))
+  (segment (start 146.872 103.048) (end 151.972 103.048) (width 0.1) (layer "F.Cu") (net 1))
+  (segment (start 143.32 102.036) (end 142.24237 102.036) (width 0.1) (layer "F.Cu") (net 2))
+  (segment (start 142.24237 102.036) (end 140.97 103.30837) (width 0.1) (layer "F.Cu") (net 2))
+  (segment (start 140.97 105.146) (end 143.32 107.496) (width 0.1) (layer "F.Cu") (net 2))
+  (segment (start 140.97 103.30837) (end 140.97 105.146) (width 0.1) (layer "F.Cu") (net 2))
+  (segment (start 141.72 103.996) (end 144.28 103.996) (width 0.1) (layer "F.Cu") (net 3))
+  (segment (start 144.28 103.996) (end 144.78 104.496) (width 0.1) (layer "F.Cu") (net 3))
+  (segment (start 144.64763 108.246) (end 142.9424 108.246) (width 0.1) (layer "F.Cu") (net 4))
+  (segment (start 140.6652 100.4508) (end 141.62 99.496) (width 0.1) (layer "F.Cu") (net 4))
+  (segment (start 147.32 105.57363) (end 144.64763 108.246) (width 0.1) (layer "F.Cu") (net 4))
+  (segment (start 142.9424 108.246) (end 140.6652 105.9688) (width 0.1) (layer "F.Cu") (net 4))
+  (segment (start 140.6652 105.9688) (end 140.6652 100.4508) (width 0.1) (layer "F.Cu") (net 4))
+  (segment (start 147.32 104.496) (end 147.32 105.57363) (width 0.1) (layer "F.Cu") (net 4))
+  (segment (start 140.3652 96.3508) (end 141.72 94.996) (width 0.1) (layer "F.Cu") (net 5))
+  (segment (start 140.3652 106.093064) (end 140.3652 96.3508) (width 0.1) (layer "F.Cu") (net 5))
+  (segment (start 145.81 108.546) (end 142.818136 108.546) (width 0.1) (layer "F.Cu") (net 5))
+  (segment (start 142.818136 108.546) (end 140.3652 106.093064) (width 0.1) (layer "F.Cu") (net 5))
+  (segment (start 149.86 104.496) (end 145.81 108.546) (width 0.1) (layer "F.Cu") (net 5))
+  (segment (start 145.751185 91.496) (end 148.3868 94.131615) (width 0.1) (layer "F.Cu") (net 6))
+  (segment (start 151.32 100.927185) (end 151.32 102.036) (width 0.1) (layer "F.Cu") (net 6))
+  (segment (start 143.32 91.496) (end 145.751185 91.496) (width 0.1) (layer "F.Cu") (net 6))
+  (segment (start 148.3868 94.131615) (end 148.3868 97.993985) (width 0.1) (layer "F.Cu") (net 6))
+  (segment (start 148.3868 97.993985) (end 151.32 100.927185) (width 0.1) (layer "F.Cu") (net 6))
+  (segment (start 151.32 99.496) (end 148.848 97.024) (width 0.1) (layer "F.Cu") (net 7))
+  (segment (start 148.848 97.024) (end 148.848 92.024) (width 0.1) (layer "F.Cu") (net 7))
+  (segment (start 148.848 92.024) (end 147.32 90.496) (width 0.1) (layer "F.Cu") (net 7))
+  (segment (start 151.32 91.496) (end 153.67 93.846) (width 0.1) (layer "F.Cu") (net 8))
+  (segment (start 152.0656 96.956) (end 151.32 96.956) (width 0.1) (layer "F.Cu") (net 8))
+  (segment (start 153.67 93.846) (end 153.67 95.3516) (width 0.1) (layer "F.Cu") (net 8))
+  (segment (start 153.67 95.3516) (end 152.0656 96.956) (width 0.1) (layer "F.Cu") (net 8))
+  (segment (start 152.92 94.996) (end 150.36 94.996) (width 0.1) (layer "F.Cu") (net 9))
+  (segment (start 150.36 94.996) (end 149.86 94.496) (width 0.1) (layer "F.Cu") (net 9))
+  (segment (start 153.02 97.224815) (end 151.303185 95.508) (width 0.1) (layer "B.Cu") (net 10))
+  (segment (start 153.02 99.496) (end 153.02 97.224815) (width 0.1) (layer "B.Cu") (net 10))
+  (segment (start 151.303185 95.508) (end 148.332 95.508) (width 0.1) (layer "B.Cu") (net 10))
+  (segment (start 148.332 95.508) (end 147.32 94.496) (width 0.1) (layer "B.Cu") (net 10))
+  (segment (start 140.8684 98.32997) (end 140.8684 102.015585) (width 0.1) (layer "B.Cu") (net 12))
+  (segment (start 143.32 96.956) (end 142.24237 96.956) (width 0.1) (layer "B.Cu") (net 12))
+  (segment (start 151.184 107.632) (end 151.32 107.496) (width 0.1) (layer "B.Cu") (net 12))
+  (segment (start 146.484815 107.632) (end 151.184 107.632) (width 0.1) (layer "B.Cu") (net 12))
+  (segment (start 140.8684 102.015585) (end 146.484815 107.632) (width 0.1) (layer "B.Cu") (net 12))
+  (segment (start 142.24237 96.956) (end 140.8684 98.32997) (width 0.1) (layer "B.Cu") (net 12))
 )
