File: pcb/motherboard/DecoderInverter.kicad_sch (KiCad schematic)
At the start: 2 parts, among them U10 74HC04, U9 74HC04

Commit message: Ver 3.0
Parts:
- removed unit 5 of U10
- removed unit 6 of U10
- removed unit 1 of U9
- removed unit 2 of U9
- removed unit 3 of U9
- removed unit 4 of U9
- added unit 2 of U8
- added unit 6 of U8
- added unit 1 of U8
- added unit 3 of U8
- added unit 4 of U8
- added unit 5 of U8
- renumbered U9 to U8, U10 to U9
Connections:
- net IN_P0: now also U8.1
- net IN_P1: now also U8.3
- net IN_P2: now also U8.5
- net IN_P3: now also U8.9
- net IN_P4: now also U8.11; no longer U9.11
- net IN_P5: now also U8.13; no longer U9.13
- net OUT_P0: now also U8.2
- net OUT_P1: now also U8.4
- net OUT_P2: now also U8.6
- net OUT_P3: now also U8.8
- net OUT_P4: now also U8.10; no longer U9.10
- net OUT_P5: now also U8.12; no longer U9.12
Other:
- moved on the sheet: U9A, U9B, U9C, U9D
