File: pcb/motherboard/NixieY.kicad_sch (KiCad schematic)
At the start: 10 parts, among them Q10 MPSA42, Q11 MPSA42, Q12 MPSA42, Q13 MPSA42, Q14 MPSA42, Q15 MPSA42, Q16 MPSA42, Q17 MPSA42, Q8 MPSA42, Q9 MPSA42

Commit message: Ver 3.0
Parts:
- renumbered Q8 to Q12, Q9 to Q13, Q10 to Q14, Q11 to Q15, Q12 to Q16, Q13 to Q17, Q14 to Q18, Q15 to Q19, Q16 to Q20, Q17 to Q21
Changed lines of the file:
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@@
   (symbol (lib_id "Transistor_BJT:MPSA42") (at 110.49 73.66 0) (unit 1)
     (in_bom yes) (on_board yes) (dnp no)
-    (property "Reference" "Q9" (at 115.3414 72.4916 0)
+    (property "Reference" "Q13" (at 115.3414 72.4916 0)
       (effects (font (size 1.27 1.27)) (justify left))
     )
@@
       (project "OpenNixie"
         (path "/2b75b537-ab0e-4c23-8f3b-4f491320330e/00000000-0000-0000-0000-00006655b5ad"
-          (reference "Q9") (unit 1)
+          (reference "Q13") (unit 1)
         )
       )
@@
   (symbol (lib_id "Transistor_BJT:MPSA42") (at 116.84 85.09 0) (unit 1)
     (in_bom yes) (on_board yes) (dnp no)
-    (property "Reference" "Q11" (at 121.6914 83.9216 0)
+    (property "Reference" "Q15" (at 121.6914 83.9216 0)
       (effects (font (size 1.27 1.27)) (justify left))
     )
@@
       (project "OpenNixie"
         (path "/2b75b537-ab0e-4c23-8f3b-4f491320330e/00000000-0000-0000-0000-00006655b5ad"
-          (reference "Q11") (unit 1)
+          (reference "Q15") (unit 1)
         )
       )
@@
   (symbol (lib_id "Transistor_BJT:MPSA42") (at 123.19 96.52 0) (unit 1)
     (in_bom yes) (on_board yes) (dnp no)
-    (property "Reference" "Q13" (at 128.0414 95.3516 0)
+    (property "Reference" "Q17" (at 128.0414 95.3516 0)
       (effects (font (size 1.27 1.27)) (justify left))
     )
@@
       (project "OpenNixie"
         (path "/2b75b537-ab0e-4c23-8f3b-4f491320330e/00000000-0000-0000-0000-00006655b5ad"
-          (reference "Q13") (unit 1)
+          (reference "Q17") (unit 1)
         )
       )
@@
   (symbol (lib_id "Transistor_BJT:MPSA42") (at 129.54 107.95 0) (unit 1)
     (in_bom yes) (on_board yes) (dnp no)
-    (property "Reference" "Q15" (at 134.3914 106.7816 0)
+    (property "Reference" "Q19" (at 134.3914 106.7816 0)
       (effects (font (size 1.27 1.27)) (justify left))
     )
@@
       (project "OpenNixie"
         (path "/2b75b537-ab0e-4c23-8f3b-4f491320330e/00000000-0000-0000-0000-00006655b5ad"
-          (reference "Q15") (unit 1)
+          (reference "Q19") (unit 1)
         )
       )
@@
   (symbol (lib_id "Transistor_BJT:MPSA42") (at 161.29 100.33 0) (unit 1)
     (in_bom yes) (on_board yes) (dnp no)
-    (property "Reference" "Q14" (at 166.1414 99.1616 0)
+    (property "Reference" "Q18" (at 166.1414 99.1616 0)
       (effects (font (size 1.27 1.27)) (justify left))
     )
@@
       (project "OpenNixie"
         (path "/2b75b537-ab0e-4c23-8f3b-4f491320330e/00000000-0000-0000-0000-00006655b5ad"
+          (reference "Q18") (unit 1)
+        )
+      )
+    )
+  )
+  (symbol (lib_id "Transistor_BJT:MPSA42") (at 154.94 88.9 0) (unit 1)
+    (in_bom yes) (on_board yes) (dnp no)
+    (property "Reference" "Q16" (at 159.7914 87.7316 0)
+      (effects (font (size 1.27 1.27)) (justify left))
+    )
+    (property "Value" "MPSA42" (at 159.7914 90.043 0)
+      (effects (font (size 1.27 1.27)) (justify left))
+    )
+    (property "Footprint" "Package_TO_SOT_THT:TO-92_Inline" (at 160.02 90.805 0)
+      (effects (font (size 1.27 1.27) italic) (justify left) hide)
+    )
+    (property "Datasheet" "http://www.onsemi.com/pub_link/Collateral/MPSA42-D.PDF" (at 154.94 88.9 0)
+      (effects (font (size 1.27 1.27)) (justify left) hide)
+    )
+    (pin "1")
+    (pin "2")
+    (pin "3")
+    (instances
+      (project "OpenNixie"
+        (path "/2b75b537-ab0e-4c23-8f3b-4f491320330e/00000000-0000-0000-0000-00006655b5ad"
+          (reference "Q16") (unit 1)
+        )
+      )
+    )
+  )
+  (symbol (lib_id "Transistor_BJT:MPSA42") (at 148.59 77.47 0) (unit 1)
+    (in_bom yes) (on_board yes) (dnp no)
+    (property "Reference" "Q14" (at 153.4414 76.3016 0)
+      (effects (font (size 1.27 1.27)) (justify left))
+    )
+    (property "Value" "MPSA42" (at 153.4414 78.613 0)
+      (effects (font (size 1.27 1.27)) (justify left))
+    )
+    (property "Footprint" "Package_TO_SOT_THT:TO-92_Inline" (at 153.67 79.375 0)
+      (effects (font (size 1.27 1.27) italic) (justify left) hide)
+    )
+    (property "Datasheet" "http://www.onsemi.com/pub_link/Collateral/MPSA42-D.PDF" (at 148.59 77.47 0)
+      (effects (font (size 1.27 1.27)) (justify left) hide)
+    )
+    (pin "1")
+    (pin "2")
+    (pin "3")
+    (instances
+      (project "OpenNixie"
+        (path "/2b75b537-ab0e-4c23-8f3b-4f491320330e/00000000-0000-0000-0000-00006655b5ad"
           (reference "Q14") (unit 1)
         )
@@
     )
   )
-  (symbol (lib_id "Transistor_BJT:MPSA42") (at 154.94 88.9 0) (unit 1)
-    (in_bom yes) (on_board yes) (dnp no)
-    (property "Reference" "Q12" (at 159.7914 87.7316 0)
-      (effects (font (size 1.27 1.27)) (justify left))
-    )
-    (property "Value" "MPSA42" (at 159.7914 90.043 0)
-      (effects (font (size 1.27 1.27)) (justify left))
-    )
-    (property "Footprint" "Package_TO_SOT_THT:TO-92_Inline" (at 160.02 90.805 0)
-      (effects (font (size 1.27 1.27) italic) (justify left) hide)
-    )
-    (property "Datasheet" "http://www.onsemi.com/pub_link/Collateral/MPSA42-D.PDF" (at 154.94 88.9 0)
+  (symbol (lib_id "Transistor_BJT:MPSA42") (at 142.24 66.04 0) (unit 1)
+    (in_bom yes) (on_board yes) (dnp no)
+    (property "Reference" "Q12" (at 147.0914 64.8716 0)
+      (effects (font (size 1.27 1.27)) (justify left))
+    )
+    (property "Value" "MPSA42" (at 147.0914 67.183 0)
+      (effects (font (size 1.27 1.27)) (justify left))
+    )
+    (property "Footprint" "Package_TO_SOT_THT:TO-92_Inline" (at 147.32 67.945 0)
+      (effects (font (size 1.27 1.27) italic) (justify left) hide)
+    )
+    (property "Datasheet" "http://www.onsemi.com/pub_link/Collateral/MPSA42-D.PDF" (at 142.24 66.04 0)
       (effects (font (size 1.27 1.27)) (justify left) hide)
     )
@@
     )
   )
-  (symbol (lib_id "Transistor_BJT:MPSA42") (at 148.59 77.47 0) (unit 1)
-    (in_bom yes) (on_board yes) (dnp no)
-    (property "Reference" "Q10" (at 153.4414 76.3016 0)
-      (effects (font (size 1.27 1.27)) (justify left))
-    )
-    (property "Value" "MPSA42" (at 153.4414 78.613 0)
-      (effects (font (size 1.27 1.27)) (justify left))
-    )
-    (property "Footprint" "Package_TO_SOT_THT:TO-92_Inline" (at 153.67 79.375 0)
-      (effects (font (size 1.27 1.27) italic) (justify left) hide)
-    )
-    (property "Datasheet" "http://www.onsemi.com/pub_link/Collateral/MPSA42-D.PDF" (at 148.59 77.47 0)
-      (effects (font (size 1.27 1.27)) (justify left) hide)
-    )
-    (pin "1")
-    (pin "2")
-    (pin "3")
-    (instances
-      (project "OpenNixie"
-        (path "/2b75b537-ab0e-4c23-8f3b-4f491320330e/00000000-0000-0000-0000-00006655b5ad"
-          (reference "Q10") (unit 1)
-        )
-      )
-    )
-  )
-  (symbol (lib_id "Transistor_BJT:MPSA42") (at 142.24 66.04 0) (unit 1)
-    (in_bom yes) (on_board yes) (dnp no)
-    (property "Reference" "Q8" (at 147.0914 64.8716 0)
-      (effects (font (size 1.27 1.27)) (justify left))
-    )
-    (property "Value" "MPSA42" (at 147.0914 67.183 0)
-      (effects (font (size 1.27 1.27)) (justify left))
-    )
-    (property "Footprint" "Package_TO_SOT_THT:TO-92_Inline" (at 147.32 67.945 0)
-      (effects (font (size 1.27 1.27) italic) (justify left) hide)
-    )
-    (property "Datasheet" "http://www.onsemi.com/pub_link/Collateral/MPSA42-D.PDF" (at 142.24 66.04 0)
-      (effects (font (size 1.27 1.27)) (justify left) hide)
-    )
-    (pin "1")
-    (pin "2")
-    (pin "3")
-    (instances
-      (project "OpenNixie"
-        (path "/2b75b537-ab0e-4c23-8f3b-4f491320330e/00000000-0000-0000-0000-00006655b5ad"
-          (reference "Q8") (unit 1)
-        )
-      )
-    )
-  )
   (symbol (lib_id "Transistor_BJT:MPSA42") (at 167.64 111.76 0) (unit 1)
     (in_bom yes) (on_board yes) (dnp no)
-    (property "Reference" "Q16" (at 172.4914 110.5916 0)
+    (property "Reference" "Q20" (at 172.4914 110.5916 0)
       (effects (font (size 1.27 1.27)) (justify left))
     )
@@
       (project "OpenNixie"
         (path "/2b75b537-ab0e-4c23-8f3b-4f491320330e/00000000-0000-0000-0000-00006655b5ad"
-          (reference "Q16") (unit 1)
+          (reference "Q20") (unit 1)
         )
       )
@@
   (symbol (lib_id "Transistor_BJT:MPSA42") (at 135.89 119.38 0) (unit 1)
     (in_bom yes) (on_board yes) (dnp no)
-    (property "Reference" "Q17" (at 140.7414 118.2116 0)
+    (property "Reference" "Q21" (at 140.7414 118.2116 0)
       (effects (font (size 1.27 1.27)) (justify left))
     )
@@
       (project "OpenNixie"
         (path "/2b75b537-ab0e-4c23-8f3b-4f491320330e/00000000-0000-0000-0000-00006655b5ad"
-          (reference "Q17") (unit 1)
+          (reference "Q21") (unit 1)
         )
       )
@@
   (symbol (lib_id "power:GND") (at 113.03 137.16 0) (unit 1)
     (in_bom yes) (on_board yes) (dnp no)
-    (property "Reference" "#PWR014" (at 113.03 143.51 0)
+    (property "Reference" "#PWR013" (at 113.03 143.51 0)
       (effects (font (size 1.27 1.27)) hide)
     )
@@
       (project "OpenNixie"
         (path "/2b75b537-ab0e-4c23-8f3b-4f491320330e/00000000-0000-0000-0000-00006655b5ad"
-          (reference "#PWR014") (unit 1)
+          (reference "#PWR013") (unit 1)
         )
         (path "/2b75b537-ab0e-4c23-8f3b-4f491320330e/00000000-0000-0000-0000-000066554687"
