File: pcb/motherboard/NixieBS.kicad_sch (KiCad schematic)
At the start: 12 parts

Commit message: Some fixes
Parts:
- renumbered R27 to R17, R28 to R18, R29 to R19, R30 to R20
Changed lines of the file:
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@@
   (symbol (lib_id "Device:R_Small") (at 160.655 47.625 0) (unit 1)
     (in_bom yes) (on_board yes) (dnp no) (fields_autoplaced)
-    (property "Reference" "R30" (at 162.1536 46.9813 0)
+    (property "Reference" "R20" (at 162.1536 46.9813 0)
       (effects (font (size 1.27 1.27)) (justify left))
     )
@@
       (project "OpenNixie"
         (path "/2b75b537-ab0e-4c23-8f3b-4f491320330e/3a351cf1-25b2-4939-9e7f-12d4a9bbcf02"
-          (reference "R30") (unit 1)
+          (reference "R20") (unit 1)
         )
       )
@@
         )
         (path "/2b75b537-ab0e-4c23-8f3b-4f491320330e/3a351cf1-25b2-4939-9e7f-12d4a9bbcf02"
-          (reference "R31") (unit 1)
+          (reference "R21") (unit 1)
         )
       )
@@
         )
         (path "/2b75b537-ab0e-4c23-8f3b-4f491320330e/3a351cf1-25b2-4939-9e7f-12d4a9bbcf02"
-          (reference "R32") (unit 1)
+          (reference "R22") (unit 1)
         )
       )
@@
   (symbol (lib_id "Device:R_Small") (at 149.225 47.625 0) (unit 1)
     (in_bom yes) (on_board yes) (dnp no) (fields_autoplaced)
-    (property "Reference" "R29" (at 150.7236 46.9813 0)
+    (property "Reference" "R19" (at 150.7236 46.9813 0)
       (effects (font (size 1.27 1.27)) (justify left))
     )
@@
       (project "OpenNixie"
         (path "/2b75b537-ab0e-4c23-8f3b-4f491320330e/3a351cf1-25b2-4939-9e7f-12d4a9bbcf02"
-          (reference "R29") (unit 1)
+          (reference "R19") (unit 1)
         )
       )
@@
   (symbol (lib_id "Device:R_Small") (at 137.795 47.625 0) (unit 1)
     (in_bom yes) (on_board yes) (dnp no) (fields_autoplaced)
-    (property "Reference" "R28" (at 139.2936 46.9813 0)
+    (property "Reference" "R18" (at 139.2936 46.9813 0)
       (effects (font (size 1.27 1.27)) (justify left))
     )
@@
       (project "OpenNixie"
         (path "/2b75b537-ab0e-4c23-8f3b-4f491320330e/3a351cf1-25b2-4939-9e7f-12d4a9bbcf02"
-          (reference "R28") (unit 1)
+          (reference "R18") (unit 1)
         )
       )
@@
         )
         (path "/2b75b537-ab0e-4c23-8f3b-4f491320330e/3a351cf1-25b2-4939-9e7f-12d4a9bbcf02"
-          (reference "R33") (unit 1)
+          (reference "R23") (unit 1)
         )
       )
@@
         )
         (path "/2b75b537-ab0e-4c23-8f3b-4f491320330e/3a351cf1-25b2-4939-9e7f-12d4a9bbcf02"
-          (reference "R34") (unit 1)
+          (reference "R24") (unit 1)
         )
       )
@@
   (symbol (lib_id "Device:R_Small") (at 126.365 47.625 0) (unit 1)
     (in_bom yes) (on_board yes) (dnp no) (fields_autoplaced)
-    (property "Reference" "R27" (at 127.8636 46.9813 0)
+    (property "Reference" "R17" (at 127.8636 46.9813 0)
       (effects (font (size 1.27 1.27)) (justify left))
     )
@@
       (project "OpenNixie"
         (path "/2b75b537-ab0e-4c23-8f3b-4f491320330e/3a351cf1-25b2-4939-9e7f-12d4a9bbcf02"
-          (reference "R27") (unit 1)
-        )
-      )
+          (reference "R17") (unit 1)
+        )
+      )
