File: pcb/motherboard/NixieSS.kicad_sch (KiCad schematic)
At the start: 30 parts

Commit message: Some fixes
Parts:
- removed R10, R11, R12, R13, R14, R15, R16, R7, R8, R9: 47k, Resistor_THT:R_Axial_DIN0204_L3.6mm_D1.6mm_P5.08mm_Horizontal, symbol Device:R_Small
