File: pcb/motherboard/OpenNixie.kicad_pcb (KiCad board)
At the start: 2 copper layers, 152 x 55 mm, 76 parts, among them J1 Conn_01x02, J10 Nixie_Conn_12P, J2 Conn_01x03, J3 Nixie_Conn_4P, J4 Conn_01x04, J5 Conn_01x03, J6 12V, J7 Nixie_Conn_12P, J8 Nixie_Conn_12P, J9 Nixie_Conn_12P, Q1 MPSA42, Q10 S8050, Q11 S8050, Q12 MPSA42, Q13 MPSA42, Q14 MPSA42, Q15 MPSA42, Q16 MPSA42, Q17 MPSA42, Q18 MPSA42, Q19 MPSA42, Q2 S8050, Q20 MPSA42, Q21 MPSA42, Q3 TK8P65W, Q4 MPSA42, Q5 MPSA42, Q6 MPSA42, Q7 MPSA42, Q8 S8050, Q9 S8050, U1 LM7805_TO220, U2 NE555P, U3 NE555P, U4 MAX1771CSA, U5 74LS138, U6 74HC595, U7 74LS138, U8 74HC04, U9 74HC04

Commit message: PCB updated
Parts:
- removed the C2 at (185.2, 79.8)
- removed the D1 at (100.2, 79.9)
- removed D3: LED_RKGB, LED_THT:LED_D5.0mm-4_RGB_Wide_Pins
- removed G1: LOGO, Nixie_Clock:Logo
- removed the J2 at (222.0, 110.0)
- removed the J3 at (150.9, 96.2)
- removed the J4 at (114.0, 72.6)
- removed the J5 at (222.0, 98.0)
- removed Q17, Q18, Q19, Q20, Q21: MPSA42, Package_TO_SOT_THT:TO-92_Inline
- removed the Q2 at (100.2, 85.8)
- removed the R3 at (137.2, 79.9)
- removed the R4 at (137.2, 83.4)
- removed REF1, REF2, REF3, REF4: MountingHole_2.2mm_M2, MountingHole:MountingHole_2.2mm_M2
- removed the U2 at (167.2, 80.1)
- removed the U3 at (124.4, 79.7)
- removed U5, U7: 74LS138, Package_DIP:DIP-16_W7.62mm
- removed U8, U9: 74HC04, Package_DIP:DIP-14_W7.62mm
- removed locked: 10k, Resistor_THT:R_Axial_DIN0204_L3.6mm_D1.6mm_P5.08mm_Horizontal
- removed locked: 150k, Resistor_THT:R_Axial_DIN0204_L3.6mm_D1.6mm_P5.08mm_Horizontal
- removed locked: 470uF, Capacitor_THT:CP_Radial_D8.0mm_P3.50mm
- removed locked: 200k, Potentiometer_THT:Potentiometer_Vishay_T73YP_Vertical
- added C1: 0.1uF, Capacitor_THT:C_Disc_D3.0mm_W2.0mm_P2.50mm, F.Cu at (105.9, 87.9)
- added G***: LOGO, Nixie_Clock:Logo, F.Cu at (183.5, 73.9)
- added H1: MountingHole, MountingHole:MountingHole_3.2mm_M3, F.Cu at (78.4, 72.8)
- added H2: MountingHole, MountingHole:MountingHole_3.2mm_M3, F.Cu at (223.4, 72.8)
- added H3: MountingHole, MountingHole:MountingHole_3.2mm_M3, F.Cu at (223.5, 120.9)
- added H4: MountingHole, MountingHole:MountingHole_3.2mm_M3, F.Cu at (78.4, 120.9)
- added NE1: Lamp_Neon, Connector_PinSocket_2.54mm:PinSocket_1x02_P2.54mm_Vertical, F.Cu at (150.9, 96.2)
- added Q3: MPSA42, Package_TO_SOT_THT:TO-92_Inline, F.Cu at (153.7, 111.3)
- added R11: 47k, Resistor_THT:R_Axial_DIN0204_L3.6mm_D1.6mm_P5.08mm_Horizontal, F.Cu at (172.7, 114.6)
- added R13: 47k, Resistor_THT:R_Axial_DIN0204_L3.6mm_D1.6mm_P5.08mm_Horizontal, F.Cu at (163.6, 80.1)
- added R22: 47k, Resistor_THT:R_Axial_DIN0204_L3.6mm_D1.6mm_P5.08mm_Horizontal, F.Cu at (210.1, 116.6)
- added R23: 47k, Resistor_THT:R_Axial_DIN0204_L3.6mm_D1.6mm_P5.08mm_Horizontal, F.Cu at (198.9, 116.6)
- added R24: 47k, Resistor_THT:R_Axial_DIN0204_L3.6mm_D1.6mm_P5.08mm_Horizontal, F.Cu at (187.5, 116.6)
- added R25: 47k, Resistor_THT:R_Axial_DIN0204_L3.6mm_D1.6mm_P5.08mm_Horizontal, F.Cu at (164.1, 116.6)
- added R26: 47k, Resistor_THT:R_Axial_DIN0204_L3.6mm_D1.6mm_P5.08mm_Horizontal, F.Cu at (175.5, 116.6)
- added R27: 47k, Resistor_THT:R_Axial_DIN0204_L3.6mm_D1.6mm_P5.08mm_Horizontal, F.Cu at (142.2, 100.1)
- added R28: 47k, Resistor_THT:R_Axial_DIN0204_L3.6mm_D1.6mm_P5.08mm_Horizontal, F.Cu at (188.7, 98.6)
- added R29: 47k, Resistor_THT:R_Axial_DIN0204_L3.6mm_D1.6mm_P5.08mm_Horizontal, F.Cu at (79.5, 115.1)
- added R30: 47k, Resistor_THT:R_Axial_DIN0204_L3.6mm_D1.6mm_P5.08mm_Horizontal, F.Cu at (161.0, 98.6)
- added R31: 47k, Resistor_THT:R_Axial_DIN0204_L3.6mm_D1.6mm_P5.08mm_Horizontal, F.Cu at (83.1, 116.6)
- added R32: 47k, Resistor_THT:R_Axial_DIN0204_L3.6mm_D1.6mm_P5.08mm_Horizontal, F.Cu at (132.3, 100.1)
- added R33: 47k, Resistor_THT:R_Axial_DIN0204_L3.6mm_D1.6mm_P5.08mm_Horizontal, F.Cu at (163.8, 100.6)
- added R34: 47k, Resistor_THT:R_Axial_DIN0204_L3.6mm_D1.6mm_P5.08mm_Horizontal, F.Cu at (192.0, 100.1)
- added R8: 47k, Resistor_THT:R_Axial_DIN0204_L3.6mm_D1.6mm_P5.08mm_Horizontal, F.Cu at (190.2, 85.0)
- added R9: 47k, Resistor_THT:R_Axial_DIN0204_L3.6mm_D1.6mm_P5.08mm_Horizontal, F.Cu at (207.3, 114.6)
- added U4: 74HC595, Package_DIP:DIP-16_W7.62mm, F.Cu at (117.9, 116.8)
- J1: value Conn_01x02 -> Jack-DC; footprint Connector_JST:JST_EH_B2B-EH-A_1x02_P2.50mm_Vertical -> Connector_BarrelJack:BarrelJack_Horizontal
- J6: value 12V -> Conn_01x05; footprint Connector_BarrelJack:BarrelJack_Horizontal -> Connector_PinHeader_2.54mm:PinHeader_1x05_P2.54mm_Vertical
- Q10, Q11, Q8, Q9: value S8050 -> MPSA42
- R1: value 47k -> 10M
- R10: value 1k -> 47k; footprint Resistor_THT:R_Axial_DIN0309_L9.0mm_D3.2mm_P12.70mm_Horizontal -> Resistor_THT:R_Axial_DIN0204_L3.6mm_D1.6mm_P5.08mm_Horizontal
- R12, R2: value 1k -> 47k
- R14, R15, R16, R17: value 36k -> 47k; footprint Resistor_THT:R_Axial_DIN0309_L9.0mm_D3.2mm_P12.70mm_Horizontal -> Resistor_THT:R_Axial_DIN0204_L3.6mm_D1.6mm_P5.08mm_Horizontal
- R18, R19, R20, R21: value 36k -> 47k
- R4: renamed from R9; value 10k -> 47k
- R7: value 150k -> 47k
- U1: value LM7805_TO220 -> AMS1117; footprint Package_TO_SOT_THT:TO-220-3_Vertical -> Package_TO_SOT_SMD:SOT-223-3_TabPin2
- moved C2 94.6 mm to (125.9, 76.2), turned to 180 degrees
- moved D1 90.9 mm to (105.4, 96.0)
- moved R20 83.2 mm to (193.5, 87.1)
- moved U3 82.5 mm to (93.0, 116.8), turned to 90 degrees
- moved R6 79.7 mm to (105.9, 76.7)
- moved C3 73.9 mm to (136.7, 76.2), turned to 180 degrees
- moved L1 73.3 mm to (131.1, 84.3)
- moved J6 68.4 mm to (83.4, 94.2), turned to 0 degrees
- moved Q2 67.9 mm to (112.5, 95.6), turned to 90 degrees
- moved U1 64.4 mm to (97.0, 83.8)
- moved R14 59.9 mm to (202.0, 85.0), turned to 90 degrees
- moved Q4 53.8 mm to (154.9, 76.9)
- moved Q12 50.1 mm to (177.0, 111.3), turned to 0 degrees
- moved Q13 49.1 mm to (84.3, 111.8), turned to 0 degrees
- moved R12 47.5 mm to (149.1, 114.6), turned to 90 degrees
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- renumbered C3 to C2, C4 to C3, C5 to C4, D2 to D1, J7 to J2, J8 to J3, J9 to J4, J10 to J5, Q3 to Q2, R8 to R3, R11 to R5, R13 to R6, U4 to U2, U6 to U3
Connections:
- C2 pad 1: +12V -> /+12v
- C3 pad 1: Net-(D2-K) -> +170v
- D1 pad 1: Net-(D2-K) -> +170v
- J1 pad 1: LIGHT_PIN -> /+12v
- J1 pad 2: SHDN_PIN -> GND
- J2 pad 0: /NIXIE_Y_P0 -> /SEG_P0
- J2 pad 1: /NIXIE_Y_P1 -> /SEG_P1
- J2 pad 2: /NIXIE_Y_P2 -> /SEG_P2
- J2 pad 3: /NIXIE_Y_P3 -> /SEG_P3
- J2 pad 4: /NIXIE_Y_P4 -> /SEG_P4
- J2 pad 5: /NIXIE_Y_P5 -> /SEG_P5
- J2 pad 6: /NIXIE_Y_P6 -> /SEG_P6
- J2 pad 7: /NIXIE_Y_P7 -> /SEG_P7
- J2 pad 8: /NIXIE_Y_P8 -> /SEG_P8
- J2 pad 9: /NIXIE_Y_P9 -> /SEG_P9
- J2 pad A: /NIXIE_X_P0 -> /BIT_P0
- J3 pad 0: /NIXIE_Y_P0 -> /SEG_P0
- J3 pad 1: /NIXIE_Y_P1 -> /SEG_P1
- J3 pad 2: /NIXIE_Y_P2 -> /SEG_P2
- J3 pad 3: /NIXIE_Y_P3 -> /SEG_P3
- J3 pad 4: /NIXIE_Y_P4 -> /SEG_P4
- J3 pad 5: /NIXIE_Y_P5 -> /SEG_P5
- J3 pad 6: /NIXIE_Y_P6 -> /SEG_P6
- J3 pad 7: /NIXIE_Y_P7 -> /SEG_P7
- J3 pad 8: /NIXIE_Y_P8 -> /SEG_P8
- J3 pad 9: /NIXIE_Y_P9 -> /SEG_P9
- J3 pad A: /NIXIE_X_P1 -> /BIT_P1
- J4 pad 0: /NIXIE_Y_P0 -> /SEG_P0
- J4 pad 1: /NIXIE_Y_P1 -> /SEG_P1
- J4 pad 2: /NIXIE_Y_P2 -> /SEG_P2
- J4 pad 3: /NIXIE_Y_P3 -> /SEG_P3
- J4 pad 4: /NIXIE_Y_P4 -> /SEG_P4
- J4 pad 5: /NIXIE_Y_P5 -> /SEG_P5
- J4 pad 6: /NIXIE_Y_P6 -> /SEG_P6
- J4 pad 7: /NIXIE_Y_P7 -> /SEG_P7
- J4 pad 8: /NIXIE_Y_P8 -> /SEG_P8
- J4 pad 9: /NIXIE_Y_P9 -> /SEG_P9
- J4 pad A: /NIXIE_X_P2 -> /BIT_P2
- J5 pad 0: /NIXIE_Y_P0 -> /SEG_P0
- J5 pad 1: /NIXIE_Y_P1 -> /SEG_P1
- J5 pad 2: /NIXIE_Y_P2 -> /SEG_P2
- J5 pad 3: /NIXIE_Y_P3 -> /SEG_P3
- J5 pad 4: /NIXIE_Y_P4 -> /SEG_P4
- J5 pad 5: /NIXIE_Y_P5 -> /SEG_P5
- J5 pad 6: /NIXIE_Y_P6 -> /SEG_P6
- J5 pad 7: /NIXIE_Y_P7 -> /SEG_P7
- J5 pad 8: /NIXIE_Y_P8 -> /SEG_P8
- J5 pad 9: /NIXIE_Y_P9 -> /SEG_P9
- J5 pad A: /NIXIE_X_P3 -> /BIT_P3
- J6 pad 1: +12V -> /SR_LATCH
- J6 pad 2: GND -> /SR_DATA
- J6 pad 3: unconnected-(J6-Pad3) -> /SR_CLOCK
- L1 pad 2: +12V -> /+12v
- Q10 pad 2: /NOT_X_P2 -> Net-(Q10-B)
- Q10 pad 3: Net-(Q10-C) -> /SEG_P7
- Q11 pad 2: /NOT_X_P3 -> Net-(Q11-B)
- Q11 pad 3: Net-(Q11-C) -> /SEG_P8
- Q12 pad 2: /NOT_Y_P0 -> Net-(Q12-B)
- Q12 pad 3: /NIXIE_Y_P0 -> /SEG_P9
- Q13 pad 2: /NOT_Y_P1 -> Net-(Q13-B)
- Q13 pad 3: /NIXIE_Y_P1 -> /BIT_P0
- Q14 pad 2: /NOT_Y_P2 -> Net-(Q14-B)
- Q14 pad 3: /NIXIE_Y_P2 -> /BIT_P1
- Q15 pad 2: /NOT_Y_P3 -> Net-(Q15-B)
- Q15 pad 3: /NIXIE_Y_P3 -> /BIT_P2
- Q16 pad 2: /NOT_Y_P4 -> Net-(Q16-B)
- Q16 pad 3: /NIXIE_Y_P4 -> /BIT_P3
- Q4 pad 3: /NIXIE_X_P0 -> /SEG_P1
- Q5 pad 3: /NIXIE_X_P1 -> /SEG_P2
- Q6 pad 2: Net-(Q10-C) -> Net-(Q6-B)
- Q6 pad 3: /NIXIE_X_P2 -> /SEG_P3
- Q7 pad 2: Net-(Q11-C) -> Net-(Q7-B)
- Q7 pad 3: /NIXIE_X_P3 -> /SEG_P4
- Q8 pad 2: /NOT_X_P0 -> Net-(Q8-B)
- Q8 pad 3: Net-(Q4-B) -> /SEG_P5
- Q9 pad 2: /NOT_X_P1 -> Net-(Q9-B)
- Q9 pad 3: Net-(Q5-B) -> /SEG_P6
- R1 pad 1: Net-(D1-A) (its old number) -> Net-(Q1-C)
- R1 pad 2: +5V -> Net-(NE1-Pad2)
- R10 pad 1: +170V -> +170v
- R10 pad 2: Net-(D2-K) -> /SEG_P7
- R12 pad 1: GND -> +170v
- R12 pad 2: Net-(D3-K) -> /SEG_P0
- R14 pad 1: +170V -> +170v
- R14 pad 2: /NIXIE_X_P1 -> /SEG_P4
- R15 pad 1: /NIXIE_X_P3 -> +170v
- R15 pad 2: +170V -> /SEG_P6
- R16 pad 1: +170V -> +170v
- R16 pad 2: /NIXIE_X_P0 -> /SEG_P8
- R17 pad 1: +170V -> /SR_SEG_P0
- R17 pad 2: /NIXIE_X_P2 -> Net-(Q3-B)
- R18 pad 1: +5V -> /SR_SEG_P1
- R18 pad 2: Net-(Q5-B) -> Net-(Q4-B)
- R19 pad 1: +5V -> /SR_SEG_P2
- R19 pad 2: Net-(Q11-C) -> Net-(Q5-B)
- R2 pad 1: Net-(U2-DIS) -> /SYMBOL
- R2 pad 2: +12V -> Net-(Q1-B)
- R20 pad 1: +5V -> /SR_SEG_P3
- R20 pad 2: Net-(Q4-B) -> Net-(Q6-B)
- R21 pad 1: +5V -> /SR_SEG_P4
- R21 pad 2: Net-(Q10-C) -> Net-(Q7-B)
- R3 pad 2: Net-(D2-K) -> +170v
- R4 pad 1: GND -> /ENABLE
- R4 pad 2: SHDN_PIN -> GND
- R7 pad 1: Net-(U2-THR) -> +170v
- R7 pad 2: Net-(U2-DIS) -> /SEG_P1
- U1 pad 1: +12V -> GND
- U1 pad 2: GND -> /+5v
- U1 pad 3: +5V -> /+12v
- U2 pad 2: +12V -> /+12v
- U2 pad 4: SHDN_PIN -> /ENABLE
- U3 pad 1: /DECODER_P1 -> /SR_SEG_P1
- U3 pad 10: +5V -> /+5v
- U3 pad 11: SR_CLK -> /SR_CLOCK
- U3 pad 12: SR_LATCH -> /SR_LATCH
- U3 pad 14: SR_DATA -> /SR_DATA
- U3 pad 15: /DECODER_P0 -> /SR_SEG_P0
- U3 pad 16: +5V -> /+5v
- U3 pad 2: /DECODER_P2 -> /SR_SEG_P2
- U3 pad 3: /DECODER_P3 -> /SR_SEG_P3
- U3 pad 4: /NOT_X_P0 -> /SR_SEG_P4
- U3 pad 5: /NOT_X_P1 -> /SR_SEG_P5
- U3 pad 6: /NOT_X_P2 -> /SR_SEG_P6
- U3 pad 7: /NOT_X_P3 -> /SR_SEG_P7
- U3 pad 9: unconnected-(U6-QH'-Pad9) -> /SR_CASCADE
Routing:
- net +5V: track 378.1 -> 0.00 mm
- net +170v: track 0.00 -> 353.3 mm, vias 0 -> 2
- net /SEG_P7: track 0.00 -> 272.6 mm
- net /SEG_P1: track 0.00 -> 268.6 mm
- net /SEG_P8: track 0.00 -> 257.1 mm
- net /SEG_P0: track 0.00 -> 248.7 mm
- net /SEG_P9: track 0.00 -> 247.4 mm, vias 0 -> 1
- net /SEG_P5: track 0.00 -> 235.6 mm
- net /SEG_P6: track 0.00 -> 234.2 mm
- net /SEG_P3: track 0.00 -> 224.6 mm
- net /SEG_P4: track 0.00 -> 219.7 mm
- net /SEG_P2: track 0.00 -> 219.4 mm
- net /NIXIE_Y_P2: track 208.8 -> 0.00 mm
- net /NIXIE_Y_P3: track 192.4 -> 0.00 mm
- net /SR_SEG_P3: track 0.00 -> 191.6 mm
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Other:
- board text added: "LCH DAT CLK +5V GND"
- board text added: "OpenNixie@ibcl.us github.com/bclswl0827/OpenNixie"
- board text removed: "locked"

Commit message: Some fixes
Parts:
- removed the G*** at (183.5, 73.9)
- removed the R10 at (184.4, 114.6)
- removed the R11 at (172.7, 114.6)
- removed the R12 at (149.1, 114.6)
- removed the R13 at (163.6, 80.1)
- removed the R14 at (202.0, 85.0)
- removed the R15 at (195.8, 114.6)
- removed the R16 at (161.0, 114.6)
- removed the R7 at (150.5, 80.2)
- removed the R8 at (190.2, 85.0)
- removed the R9 at (207.3, 114.6)
- added G***: LOGO, Nixie_Clock:Icon_OpenSource, F.Cu at (147.5, 77.0)
- added G***: Icon_Risk, Nixie_Clock:Icon_Risk, F.Cu at (183.5, 77.0)
- R1: value 10M -> 1M
- moved R8 66.0 mm to (216.0, 103.3)
- moved Q4 65.6 mm to (217.0, 98.0)
- moved R9 50.1 mm to (216.0, 91.3)
- moved Q5 49.9 mm to (217.0, 86.1)
- moved Q6 33.5 mm to (210.8, 111.1)
- moved R10 33.4 mm to (209.5, 116.4)
- moved R11 29.7 mm to (200.8, 116.5)
- moved Q7 29.7 mm to (202.0, 111.1)
- moved Q8 18.3 mm to (193.2, 111.1)
- moved R12 18.3 mm to (191.7, 116.5)
- moved Q9 15.8 mm to (184.4, 111.1)
- moved R13 15.8 mm to (183.1, 116.5)
- moved R14 13.2 mm to (174.3, 116.5)
- moved Q10 13.2 mm to (175.6, 111.2)
- moved Q12 9.83 mm to (167.2, 111.2)
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- renumbered R20 to R10, R21 to R11, R22 to R12, R23 to R13, R24 to R14, R25 to R15, R26 to R16, R27 to R17, R28 to R18, R29 to R19, R30 to R20, R31 to R21, R32 to R22, R33 to R23, R34 to R24, R17 to R7, R18 to R8, R19 to R9
Routing:
- net +170v: track 353.3 -> 191.7 mm
- net /SR_SEG_P3: track 191.6 -> 114.2 mm
- net /SR_SEG_P2: track 88.1 -> 153.9 mm, vias 1 -> 0
- net /SR_SEG_P1: track 84.7 -> 136.1 mm, vias 1 -> 0
- net /SR_SEG_P4: track 153.7 -> 102.5 mm
- net /SEG_P1: track 268.6 -> 234.9 mm, vias 0 -> 1
- net /SEG_P9: track 247.4 -> 276.0 mm
- net /SEG_P2: track 219.4 -> 195.0 mm, vias 0 -> 1
- net /SEG_P7: track 272.6 -> 291.1 mm, vias 0 -> 1
- net /SR_SEG_P5: track 109.2 -> 91.9 mm
- net /SR_SEG_P6: track 96.0 -> 80.3 mm
- net /SR_SEG_P7: track 81.6 -> 68.4 mm
- net /SEG_P8: track 257.1 -> 268.7 mm, vias 0 -> 2
- net /SR_SEG_P9: track 59.6 -> 50.1 mm
- net /SEG_P6: track 234.2 -> 240.9 mm
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Other:
- board text added: "HIGH VOLTAGE DANGER DO NOT TOUCH DURING OPERATION"
