File: circuit/motherboard/NixieBS.kicad_sch (KiCad schematic)
At the start: 12 parts

Commit message: Some integration works
Parts:
- R20: renamed from R17; value 47k -> 20k; footprint Resistor_THT:R_Axial_DIN0204_L3.6mm_D1.6mm_P5.08mm_Horizontal -> Resistor_THT:R_Axial_DIN0207_L6.3mm_D2.5mm_P10.16mm_Horizontal
- R21: renamed from R18; value 47k -> 20k; footprint Resistor_THT:R_Axial_DIN0204_L3.6mm_D1.6mm_P5.08mm_Horizontal -> Resistor_THT:R_Axial_DIN0207_L6.3mm_D2.5mm_P10.16mm_Horizontal
- R22: renamed from R19; value 47k -> 20k; footprint Resistor_THT:R_Axial_DIN0204_L3.6mm_D1.6mm_P5.08mm_Horizontal -> Resistor_THT:R_Axial_DIN0207_L6.3mm_D2.5mm_P10.16mm_Horizontal
- R23: renamed from R20; value 47k -> 20k; footprint Resistor_THT:R_Axial_DIN0204_L3.6mm_D1.6mm_P5.08mm_Horizontal -> Resistor_THT:R_Axial_DIN0207_L6.3mm_D2.5mm_P10.16mm_Horizontal
- R? (x4): footprint Resistor_THT:R_Axial_DIN0204_L3.6mm_D1.6mm_P5.08mm_Horizontal -> Resistor_THT:R_Axial_DIN0204_L3.6mm_D1.6mm_P7.62mm_Horizontal
Changed lines of the file:
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@@
   (symbol (lib_id "Device:R_Small") (at 160.655 47.625 0) (unit 1)
     (in_bom yes) (on_board yes) (dnp no) (fields_autoplaced)
-    (property "Reference" "R20" (at 162.1536 46.9813 0)
-      (effects (font (size 1.27 1.27)) (justify left))
-    )
-    (property "Value" "47k" (at 162.1536 48.9023 0)
-      (effects (font (size 1.27 1.27)) (justify left))
-    )
-    (property "Footprint" "Resistor_THT:R_Axial_DIN0204_L3.6mm_D1.6mm_P5.08mm_Horizontal" (at 160.655 47.625 0)
+    (property "Reference" "R23" (at 162.1536 46.9813 0)
+      (effects (font (size 1.27 1.27)) (justify left))
+    )
+    (property "Value" "20k" (at 162.1536 48.9023 0)
+      (effects (font (size 1.27 1.27)) (justify left))
+    )
+    (property "Footprint" "Resistor_THT:R_Axial_DIN0207_L6.3mm_D2.5mm_P10.16mm_Horizontal" (at 160.655 47.625 0)
       (effects (font (size 1.27 1.27)) hide)
     )
@@
       (project "OpenNixie"
         (path "/2b75b537-ab0e-4c23-8f3b-4f491320330e/3a351cf1-25b2-4939-9e7f-12d4a9bbcf02"
-          (reference "R20") (unit 1)
+          (reference "R23") (unit 1)
         )
       )
@@
       (effects (font (size 1.27 1.27)))
     )
-    (property "Footprint" "Resistor_THT:R_Axial_DIN0204_L3.6mm_D1.6mm_P5.08mm_Horizontal" (at 102.87 90.17 0)
+    (property "Footprint" "Resistor_THT:R_Axial_DIN0204_L3.6mm_D1.6mm_P7.62mm_Horizontal" (at 102.87 90.17 0)
       (effects (font (size 1.27 1.27)) hide)
     )
@@
         )
         (path "/2b75b537-ab0e-4c23-8f3b-4f491320330e/3a351cf1-25b2-4939-9e7f-12d4a9bbcf02"
-          (reference "R21") (unit 1)
+          (reference "R24") (unit 1)
         )
       )
@@
       (effects (font (size 1.27 1.27)))
     )
-    (property "Footprint" "Resistor_THT:R_Axial_DIN0204_L3.6mm_D1.6mm_P5.08mm_Horizontal" (at 102.87 97.79 0)
+    (property "Footprint" "Resistor_THT:R_Axial_DIN0204_L3.6mm_D1.6mm_P7.62mm_Horizontal" (at 102.87 97.79 0)
       (effects (font (size 1.27 1.27)) hide)
     )
@@
         )
         (path "/2b75b537-ab0e-4c23-8f3b-4f491320330e/3a351cf1-25b2-4939-9e7f-12d4a9bbcf02"
-          (reference "R22") (unit 1)
+          (reference "R25") (unit 1)
         )
       )
@@
   (symbol (lib_id "Device:R_Small") (at 149.225 47.625 0) (unit 1)
     (in_bom yes) (on_board yes) (dnp no) (fields_autoplaced)
-    (property "Reference" "R19" (at 150.7236 46.9813 0)
-      (effects (font (size 1.27 1.27)) (justify left))
-    )
-    (property "Value" "47k" (at 150.7236 48.9023 0)
-      (effects (font (size 1.27 1.27)) (justify left))
-    )
-    (property "Footprint" "Resistor_THT:R_Axial_DIN0204_L3.6mm_D1.6mm_P5.08mm_Horizontal" (at 149.225 47.625 0)
+    (property "Reference" "R22" (at 150.7236 46.9813 0)
+      (effects (font (size 1.27 1.27)) (justify left))
+    )
+    (property "Value" "20k" (at 150.7236 48.9023 0)
+      (effects (font (size 1.27 1.27)) (justify left))
+    )
+    (property "Footprint" "Resistor_THT:R_Axial_DIN0207_L6.3mm_D2.5mm_P10.16mm_Horizontal" (at 149.225 47.625 0)
       (effects (font (size 1.27 1.27)) hide)
     )
@@
       (project "OpenNixie"
         (path "/2b75b537-ab0e-4c23-8f3b-4f491320330e/3a351cf1-25b2-4939-9e7f-12d4a9bbcf02"
-          (reference "R19") (unit 1)
+          (reference "R22") (unit 1)
         )
       )
@@
   (symbol (lib_id "Device:R_Small") (at 137.795 47.625 0) (unit 1)
     (in_bom yes) (on_board yes) (dnp no) (fields_autoplaced)
-    (property "Reference" "R18" (at 139.2936 46.9813 0)
-      (effects (font (size 1.27 1.27)) (justify left))
-    )
-    (property "Value" "47k" (at 139.2936 48.9023 0)
-      (effects (font (size 1.27 1.27)) (justify left))
-    )
-    (property "Footprint" "Resistor_THT:R_Axial_DIN0204_L3.6mm_D1.6mm_P5.08mm_Horizontal" (at 137.795 47.625 0)
+    (property "Reference" "R21" (at 139.2936 46.9813 0)
+      (effects (font (size 1.27 1.27)) (justify left))
+    )
+    (property "Value" "20k" (at 139.2936 48.9023 0)
+      (effects (font (size 1.27 1.27)) (justify left))
+    )
+    (property "Footprint" "Resistor_THT:R_Axial_DIN0207_L6.3mm_D2.5mm_P10.16mm_Horizontal" (at 137.795 47.625 0)
       (effects (font (size 1.27 1.27)) hide)
     )
@@
       (project "OpenNixie"
         (path "/2b75b537-ab0e-4c23-8f3b-4f491320330e/3a351cf1-25b2-4939-9e7f-12d4a9bbcf02"
-          (reference "R18") (unit 1)
+          (reference "R21") (unit 1)
         )
       )
@@
       (effects (font (size 1.27 1.27)))
     )
-    (property "Footprint" "Resistor_THT:R_Axial_DIN0204_L3.6mm_D1.6mm_P5.08mm_Horizontal" (at 102.87 105.41 0)
+    (property "Footprint" "Resistor_THT:R_Axial_DIN0204_L3.6mm_D1.6mm_P7.62mm_Horizontal" (at 102.87 105.41 0)
       (effects (font (size 1.27 1.27)) hide)
     )
@@
         )
         (path "/2b75b537-ab0e-4c23-8f3b-4f491320330e/3a351cf1-25b2-4939-9e7f-12d4a9bbcf02"
-          (reference "R23") (unit 1)
+          (reference "R26") (unit 1)
         )
       )
@@
       (effects (font (size 1.27 1.27)))
     )
-    (property "Footprint" "Resistor_THT:R_Axial_DIN0204_L3.6mm_D1.6mm_P5.08mm_Horizontal" (at 102.87 113.03 0)
+    (property "Footprint" "Resistor_THT:R_Axial_DIN0204_L3.6mm_D1.6mm_P7.62mm_Horizontal" (at 102.87 113.03 0)
       (effects (font (size 1.27 1.27)) hide)
     )
@@
         )
         (path "/2b75b537-ab0e-4c23-8f3b-4f491320330e/3a351cf1-25b2-4939-9e7f-12d4a9bbcf02"
-          (reference "R24") (unit 1)
+          (reference "R27") (unit 1)
         )
       )
@@
   (symbol (lib_id "Device:R_Small") (at 126.365 47.625 0) (unit 1)
     (in_bom yes) (on_board yes) (dnp no) (fields_autoplaced)
-    (property "Reference" "R17" (at 127.8636 46.9813 0)
-      (effects (font (size 1.27 1.27)) (justify left))
-    )
-    (property "Value" "47k" (at 127.8636 48.9023 0)
-      (effects (font (size 1.27 1.27)) (justify left))
-    )
-    (property "Footprint" "Resistor_THT:R_Axial_DIN0204_L3.6mm_D1.6mm_P5.08mm_Horizontal" (at 126.365 47.625 0)
+    (property "Reference" "R20" (at 127.8636 46.9813 0)
+      (effects (font (size 1.27 1.27)) (justify left))
+    )
+    (property "Value" "20k" (at 127.8636 48.9023 0)
+      (effects (font (size 1.27 1.27)) (justify left))
+    )
+    (property "Footprint" "Resistor_THT:R_Axial_DIN0207_L6.3mm_D2.5mm_P10.16mm_Horizontal" (at 126.365 47.625 0)
       (effects (font (size 1.27 1.27)) hide)
     )
@@
       (project "OpenNixie"
         (path "/2b75b537-ab0e-4c23-8f3b-4f491320330e/3a351cf1-25b2-4939-9e7f-12d4a9bbcf02"
-          (reference "R17") (unit 1)
+          (reference "R20") (unit 1)
         )
       )
@@
         )
         (path "/2b75b537-ab0e-4c23-8f3b-4f491320330e/3a351cf1-25b2-4939-9e7f-12d4a9bbcf02"
-          (reference "#PWR011") (unit 1)
-        )
-      )
+          (reference "#PWR017") (unit 1)
+        )
+      )
