File: circuit/motherboard/NixieSS.kicad_sch (KiCad schematic)
At the start: 20 parts

Commit message: Some integration works
Parts:
- R? (x10): footprint Resistor_THT:R_Axial_DIN0204_L3.6mm_D1.6mm_P5.08mm_Horizontal -> Resistor_THT:R_Axial_DIN0204_L3.6mm_D1.6mm_P7.62mm_Horizontal
