File: circuit/holder/QS-30/QS-30.kicad_sch (KiCad schematic)
At the start: 2 parts, among them J1 Nixie_Conn_12P

Commit message: Update schematics
Parts:
- removed NX1: QS27-1, Nixie_Clock:QS30-1, symbol Nixie_Clock:QS27-1
- added NX1: QS30-1, Nixie_Clock:QS30-1, symbol Nixie_Clock:QS30-1
Connections:
- net P0: now also NX1.0
- net P1: now also NX1.1
- net P2: now also NX1.2
- net P3: now also NX1.3
- net P4: now also NX1.4
- net P5: now also NX1.5
- net P6: now also NX1.6
- net P7: now also NX1.7
- net P8: now also NX1.8
- net P9: now also NX1.9
- net PA: now also NX1.A
Changed lines of the file:
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@@
     )
   )
-  (symbol (lib_id "Nixie_Clock:QS27-1") (at 189.23 96.52 0) (unit 1)
+  (symbol (lib_id "Nixie_Clock:QS30-1") (at 189.23 96.52 0) (unit 1)
     (in_bom yes) (on_board yes) (dnp no) (fields_autoplaced)
     (property "Reference" "NX1" (at 187.96 77.1907 0)
       (effects (font (size 1.143 1.143)))
     )
-    (property "Value" "QS27-1" (at 195.58 99.06 0)
+    (property "Value" "QS30-1" (at 195.58 99.06 0)
       (effects (font (size 1.143 1.143)) (justify left bottom) hide)
     )
